File: ee326task5.kicad_pcb (KiCad board)
At the start: 2 copper layers, 0 parts

Commit message: Started PCB Board
Parts:
- added C1: 1uF, Capacitor_SMD:C_0805_2012Metric, F.Cu at (27.9, 76.2)
- added C10: 0.1uF, Capacitor_SMD:C_0805_2012Metric, F.Cu at (72.7, 104.1)
- added C11: 0.1uF, Capacitor_SMD:C_0805_2012Metric, F.Cu at (83.8, 85.4)
- added C12: 4.7uF, Capacitor_SMD:C_0805_2012Metric, F.Cu at (83.8, 88.4)
- added C13: 0.1uF, Capacitor_SMD:C_0805_2012Metric, F.Cu at (73.7, 111.8)
- added C2: 1uF, Capacitor_SMD:C_0805_2012Metric, F.Cu at (34.0, 76.2)
- added C3: 1uF, Capacitor_SMD:C_0805_2012Metric, F.Cu at (82.9, 116.8)
- added C4: 0.1uF, Capacitor_SMD:C_0805_2012Metric, F.Cu at (74.9, 94.5)
- added C5: 18pF, Capacitor_SMD:C_0805_2012Metric, F.Cu at (41.0, 63.5)
- added C6: 18pF, Capacitor_SMD:C_0805_2012Metric, F.Cu at (46.1, 63.5)
- added C7: 0.1uF, Capacitor_SMD:C_0805_2012Metric, F.Cu at (77.8, 114.3)
- added C8: 0.1uF, Capacitor_SMD:C_0805_2012Metric, F.Cu at (76.2, 106.7)
- added C9: 0.1uF, Capacitor_SMD:C_0805_2012Metric, F.Cu at (83.8, 99.1)
- added J1: 694106106102, 694106106102:694106106102, F.Cu at (30.2, 94.0)
- added J2: Conn_01x03, Connector_PinHeader_2.54mm:PinHeader_1x03_P2.54mm_Vertical, F.Cu at (69.6, 91.4)
- added J3: Conn_01x03, Connector_PinHeader_2.54mm:PinHeader_1x03_P2.54mm_Vertical, F.Cu at (66.0, 91.4)
- added J4: Conn_01x03, Connector_PinHeader_2.54mm:PinHeader_1x03_P2.54mm_Vertical, F.Cu at (34.1, 71.1)
- added J5: Conn_01x03, Connector_PinHeader_2.54mm:PinHeader_1x03_P2.54mm_Vertical, F.Cu at (30.5, 71.1)
- added J6: 2-1734592-4, 2_1734592_4:TE_2-1734592-4, F.Cu at (49.0, 96.5)
- added L1: 10uH, Inductor_SMD:L_0805_2012Metric, F.Cu at (120.8, 75.0)
- added LED1: YELLOW, LED_SMD:LED_0603_1608Metric, F.Cu at (61.4, 54.8)
- added LED2: GREEN, LED_SMD:LED_0603_1608Metric, F.Cu at (66.5, 54.8)
- added LED3: RED, LED_SMD:LED_0603_1608Metric, F.Cu at (71.5, 54.8)
- added LED4: BLUE, LED_SMD:LED_0603_1608Metric, F.Cu at (129.5, 63.5)
- added R1: 330R, Resistor_SMD:R_0805_2012Metric, F.Cu at (61.4, 60.0)
- added R2: 330R, Resistor_SMD:R_0805_2012Metric, F.Cu at (66.5, 60.0)
- added R3: 330R, Resistor_SMD:R_0805_2012Metric, F.Cu at (71.5, 60.0)
- added R4: 330R, Resistor_SMD:R_0805_2012Metric, F.Cu at (123.5, 63.5)
- added R5: 10k, Resistor_SMD:R_0805_2012Metric, F.Cu at (117.4, 69.2)
- added R6: 10k, Resistor_SMD:R_0805_2012Metric, F.Cu at (117.4, 72.2)
- added R7: 1k, Resistor_SMD:R_0805_2012Metric, F.Cu at (121.8, 66.3)
- added R8: 1k, Resistor_SMD:R_0805_2012Metric, F.Cu at (121.8, 69.2)
- added R9: 1R0, Resistor_SMD:R_0805_2012Metric, F.Cu at (121.8, 72.2)
- added SW1: MCU_RESET, EE326_PUSH_BTN:pushbutton, F.Cu at (38.1, 55.9)
- added SW2: PROVISIONING, EE326_PUSH_BTN:pushbutton, F.Cu at (30.5, 55.9)
- added SW3: WIFI_RESET, EE326_PUSH_BTN:pushbutton, F.Cu at (116.8, 55.9)
- added SW4: IO0, EE326_PUSH_BTN:pushbutton, F.Cu at (58.4, 91.4)
- added U1: ATSAM4S8BA-AU, ATSAM4S8BA_AU:QFP50P1200X1200X160-64N, F.Cu at (48.3, 86.4)
- added U2: LDL1117S30R, LDL1117S30R:SOT230P700X180-4N, F.Cu at (38.1, 81.3)
- added U3: ESP32-WROOM-32, RF_Module:ESP32-WROOM-32E, F.Cu at (69.2, 73.7)
- added Y1: ABM7-12.000MHZ-D2Y-T, ABM7_12_000MHZ_D2Y_T:XTAL_ABM7-12.000MHZ-D2Y-T, F.Cu at (43.6, 68.6)
