File: ee326task5.kicad_sch (KiCad schematic)
At the start: 41 parts, among them J1 694106106102, J2 Conn_01x03, J3 Conn_01x03, J4 Conn_01x03, J5 Conn_01x03, J6 2-1734592-4, SW1 MCU_RESET, SW2 PROVISIONING, SW3 WIFI_RESET, SW4 IO0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

Commit message: Started PCB Board
Parts:
- C1, C10, C11, C12, C13, C2, C3, C4, C5, C6, C7, C8, C9: footprint (none) -> Capacitor_SMD:C_0805_2012Metric
- J6: footprint 2-1734592-4:TE_2-1734592-4 -> 2_1734592_4:TE_2-1734592-4
- L1: footprint (none) -> Inductor_SMD:L_0805_2012Metric
- R5, R6, R7, R8, R9: footprint (none) -> Resistor_SMD:R_0805_2012Metric
- U1: footprint ATSAM4S8BA-AU:QFP50P1200X1200X160-64N -> ATSAM4S8BA_AU:QFP50P1200X1200X160-64N
- Y1: footprint ABM7-12.000MHZ-D2Y-T:XTAL_ABM7-12.000MHZ-D2Y-T -> ABM7_12_000MHZ_D2Y_T:XTAL_ABM7-12.000MHZ-D2Y-T
Connections:
- net MCU_RX: now also U1.35 (PA5/PGMRDY)
- net MCU_TX: now also U1.34 (PA6/PGMNOE)
- net VDD3V0: no longer U2.4 (VOUT__1)
Other:
- company: (none) -> Northwestern University
- title: (none) -> EE326 Webcam Board
Changed lines of the file:
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@@
 	(generator_version "9.0")
 	(paper "A4")
-	(junction
-		(at 90.17 43.18)
-		(diameter 0)
-		(color 0 0 0 0)
+	(title_block
+		(title "EE326 Webcam Board")
+		(date "2026-02-15")
+		(rev "1")
+		(company "Northwestern University")
 	)
 	(junction
-		(at 163.83 22.86)
+		(at 90.17 43.18)
 		(diameter 0)
 		(color 0 0 0 0)
@@
 	)
 	(junction
-		(at 246.38 54.61)
-		(diameter 0)
-		(color 0 0 0 0)
-	)
-	(junction
 		(at 67.31 143.51)
 		(diameter 0)
@@
 	(wire
 		(pts
-			(xy 242.57 57.15) (xy 246.38 57.15)
-		)
-		(stroke
-			(width 0)
-			(type default)
-		)
-	)
-	(wire
-		(pts
 			(xy 241.3 114.3) (xy 248.92 114.3)
 		)
@@
 	(wire
 		(pts
-			(xy 246.38 57.15) (xy 246.38 54.61)
-		)
-		(stroke
-			(width 0)
-			(type default)
-		)
-	)
-	(wire
-		(pts
 			(xy 76.2 30.48) (xy 90.17 30.48)
 		)
@@
 	(wire
 		(pts
-			(xy 163.83 24.13) (xy 163.83 22.86)
-		)
-		(stroke
-			(width 0)
-			(type default)
-		)
-	)
-	(wire
-		(pts
 			(xy 241.3 132.08) (xy 248.92 132.08)
 		)
@@
 	(wire
 		(pts
-			(xy 246.38 54.61) (xy 252.73 54.61)
+			(xy 242.57 54.61) (xy 252.73 54.61)
 		)
 		(stroke
@@
 	(wire
 		(pts
-			(xy 132.08 170.18) (xy 137.16 170.18)
+			(xy 163.83 19.05) (xy 163.83 22.86)
 		)
 		(stroke
@@
 	(wire
 		(pts
-			(xy 90.17 38.1) (xy 99.06 38.1)
+			(xy 132.08 170.18) (xy 137.16 170.18)
 		)
 		(stroke
@@
 	(wire
 		(pts
-			(xy 157.48 107.95) (xy 152.4 107.95)
+			(xy 90.17 38.1) (xy 99.06 38.1)
 		)
 		(stroke
@@
 	(wire
 		(pts
-			(xy 242.57 54.61) (xy 246.38 54.61)
+			(xy 157.48 107.95) (xy 152.4 107.95)
 		)
 		(stroke
@@
 	(wire
 		(pts
+			(xy 100.33 71.12) (xy 90.17 71.12)
+		)
+		(stroke
+			(width 0)
+			(type default)
+		)
+	)
+	(wire
+		(pts
 			(xy 13.97 86.36) (xy 24.13 86.36)
 		)
@@
 	(wire
 		(pts
+			(xy 100.33 73.66) (xy 90.17 73.66)
+		)
+		(stroke
+			(width 0)
+			(type default)
+		)
+	)
+	(wire
+		(pts
 			(xy 80.01 143.51) (xy 78.74 143.51)
 		)
@@
 	(wire
 		(pts
-			(xy 163.83 22.86) (xy 163.83 19.05)
-		)
-		(stroke
-			(width 0)
-			(type default)
-		)
-	)
-	(wire
-		(pts
 			(xy 90.17 55.88) (xy 95.25 55.88)
 		)
@@
 		)
 	)
+	(label "MCU_TX"
+		(at 100.33 73.66 180)
+		(effects
+			(font
+				(size 1.27 1.27)
+			)
+			(justify right bottom)
+		)
+	)
 	(label "D6"
 		(at 95.25 63.5 180)
@@
 		)
 	)
+	(label "MCU_RX"
+		(at 100.33 71.12 180)
+		(effects
+			(font
+				(size 1.27 1.27)
+			)
+			(justify right bottom)
+		)
+	)
 	(label "VDD3V0"
 		(at 31.75 135.89 180)
@@
 			)
 		)
-		(property "Footprint" ""
+		(property "Footprint" "Capacitor_SMD:C_0805_2012Metric"
 			(at 76.2 32.0548 0)
 			(effects
@@
 			)
 		)
-		(property "Footprint" ""
+		(property "Footprint" "Capacitor_SMD:C_0805_2012Metric"
 			(at 76.2 29.5148 0)
 			(effects
@@
 			)
 		)
-		(property "Footprint" ""
+		(property "Footprint" "Inductor_SMD:L_0805_2012Metric"
 			(at 102.87 35.56 0)
 			(effects
@@
 			)
 		)
-		(property "Footprint" ""
+		(property "Footprint" "Capacitor_SMD:C_0805_2012Metric"
 			(at 133.0452 26.67 0)
 			(effects
@@
 			)
 		)
-		(property "Footprint" ""
+		(property "Footprint" "Capacitor_SMD:C_0805_2012Metric"
 			(at 76.2 39.6748 0)
 			(effects
@@
 			)
 		)
-		(property "Footprint" "ATSAM4S8BA-AU:QFP50P1200X1200X160-64N"
+		(property "Footprint" "ATSAM4S8BA_AU:QFP50P1200X1200X160-64N"
 			(at 57.15 66.04 0)
 			(effects
@@
 			)
 		)
-		(property "Footprint" ""
+		(property "Footprint" "Resistor_SMD:R_0805_2012Metric"
 			(at 141.732 22.86 90)
 			(effects
@@
 			)
 		)
-		(property "Footprint" ""
+		(property "Footprint" "Resistor_SMD:R_0805_2012Metric"
 			(at 100.33 62.738 90)
 			(effects
@@
 			)
 		)
-		(property "Footprint" ""
+		(property "Footprint" "Resistor_SMD:R_0805_2012Metric"
 			(at 29.972 142.24 90)
 			(effects
@@
 			)
 		)
-		(property "Footprint" "2-1734592-4:TE_2-1734592-4"
+		(property "Footprint" "2_1734592_4:TE_2-1734592-4"
 			(at 261.62 119.38 0)
 			(effects
@@
 			)
 		)
-		(property "Footprint" ""
+		(property "Footprint" "Capacitor_SMD:C_0805_2012Metric"
 			(at 66.3448 146.05 0)
 			(effects
@@
 			)
 		)
-		(property "Footprint" "ABM7-12.000MHZ-D2Y-T:XTAL_ABM7-12.000MHZ-D2Y-T"
+		(property "Footprint" "ABM7_12_000MHZ_D2Y_T:XTAL_ABM7-12.000MHZ-D2Y-T"
 			(at 73.66 143.51 0)
 			(effects
@@
 			)
 		)
-		(property "Footprint" ""
+		(property "Footprint" "Resistor_SMD:R_0805_2012Metric"
 			(at 100.33 70.358 90)
 			(effects
@@
 			)
 		)
-		(property "Footprint" ""
+		(property "Footprint" "Capacitor_SMD:C_0805_2012Metric"
 			(at 253.6952 62.23 0)
 			(effects
@@
 			)
 		)
-		(property "Footprint" ""
+		(property "Footprint" "Capacitor_SMD:C_0805_2012Metric"
 			(at 79.0448 146.05 0)
 			(effects
@@
 			)
 		)
-		(property "Footprint" ""
+		(property "Footprint" "Capacitor_SMD:C_0805_2012Metric"
 			(at 37.7952 181.61 0)
 			(effects
@@
 			)
 		)
-		(property "Footprint" ""
+		(property "Footprint" "Capacitor_SMD:C_0805_2012Metric"
 			(at 76.2 37.1348 0)
 			(effects
@@
 			)
 		)
-		(property "Footprint" ""
+		(property "Footprint" "Resistor_SMD:R_0805_2012Metric"
 			(at 106.172 39.37 90)
 			(effects
@@
 			)
 		)
-		(property "Footprint" ""
+		(property "Footprint" "Capacitor_SMD:C_0805_2012Metric"
 			(at 108.9152 50.8 0)
 			(effects
@@
 			)
 		)
-		(property "Footprint" ""
+		(property "Footprint" "Capacitor_SMD:C_0805_2012Metric"
 			(at 76.2 42.2148 0)
 			(effects
@@
 			)
 		)
-		(property "Footprint" ""
+		(property "Footprint" "Capacitor_SMD:C_0805_2012Metric"
 			(at 207.9752 62.23 0)
 			(effects
@@
 			)
 		)
-		(property "Footprint" ""
+		(property "Footprint" "Capacitor_SMD:C_0805_2012Metric"
 			(at 119.0752 43.18 0)
 			(effects

Commit message: fixed schematic errors
Connections:
- net DEBUG_RX: now also U3.34 (RXD0/IO3); no longer U3.35 (TXD0/IO1)
- net DEBUG_TX: now also U3.35 (TXD0/IO1); no longer U3.34 (RXD0/IO3)
- net VDD1V2: now also C11.2, U1.8 (VDDOUT)
- net VDD3V0: now also U2.4 (VOUT__1)
- no-connect marks 0 -> 43
Other:
- moved on the sheet: C2, C3, J1, J2, J3, J4, J5, LED1, LED2, LED3, LED4, R1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

Commit message: routing
Connections:
- net GND: now also C10.2; no longer C10.1
- net VDD1V2: now also C10.1; no longer C10.2
Other:
- moved on the sheet: C10
Changed lines of the file:
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@@
 	(symbol
 		(lib_id "Device:C")
-		(at 72.39 40.64 90)
-		(unit 1)
-		(exclude_from_sim no)
-		(in_bom yes)
-		(on_board yes)
-		(dnp no)
-		(fields_autoplaced yes)
+		(at 72.39 40.64 270)
+		(mirror x)
+		(unit 1)
+		(exclude_from_sim no)
+		(in_bom yes)
+		(on_board yes)
+		(dnp no)
 		(property "Reference" "C10"
 			(at 72.39 33.02 90)
@@
 		)
 		(property "Footprint" "Capacitor_SMD:C_0805_2012Metric"
-			(at 76.2 39.6748 0)
+			(at 68.58 39.6748 0)
 			(effects
 				(font
@@
 					(size 1.27 1.27)
 				)
-				(justify left)
-			)
-		)
+				(justify right)
+			)
+		)
